File: Milo_Ringlight/KiCad/Milo_RingLight/Milo_RingLight.kicad_pcb (KiCad board)
At the start: 2 copper layers, 85 x 81 mm, 16 parts, among them J1 Barrel_Jack_MountingPin, J2 MountingHole, J3 MountingHole, J4 MountingHole, J5 MountingHole, J6 Power Connector

Commit message: Champion Idiot. Forgot to generate Drills.
Other:
- outline, holes or cut-outs redrawn
- board text added: "Millennium Machines Milo LED Ring Light V1.1"
- board text removed: "Millennium Machines Milo LED Ring Light V1"
Changed lines of the file:
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@@
   (gr_line (start 112.499312 55.100003) (end 112.5 55.1)
     (stroke (width 0.2) (type solid)) (layer "Edge.Cuts"))
-  (gr_circle (center 32.500343 97.6) (end 34.600343 97.6)
-    (stroke (width 0.2) (type solid)) (fill none) (layer "Edge.Cuts"))
-  (gr_circle (center 107.5 82.6) (end 109.6 82.6)
-    (stroke (width 0.2) (type solid)) (fill none) (layer "Edge.Cuts"))
   (gr_arc (start 92.275963 28.104047) (mid 101.659586 40.177847) (end 105 55.1)
     (stroke (width 0.2) (type solid)) (layer "Edge.Cuts"))
@@
   (gr_line (start 112.5 56.341751) (end 112.481855 56.341751)
     (stroke (width 0.2) (type solid)) (layer "Edge.Cuts"))
-  (gr_circle (center 32.500343 82.6) (end 34.600343 82.6)
-    (stroke (width 0.2) (type solid)) (fill none) (layer "Edge.Cuts"))
   (gr_arc (start 31.500343 102.6) (mid 28.671916 101.428427) (end 27.500343 98.6)
     (stroke (width 0.2) (type solid)) (layer "Edge.Cuts"))
@@
   (gr_line (start 48.272125 24.069378) (end 47.409169 22.83695)
     (stroke (width 0.2) (type solid)) (layer "Edge.Cuts"))
-  (gr_circle (center 107.5 97.6) (end 109.6 97.6)
-    (stroke (width 0.2) (type solid)) (fill none) (layer "Edge.Cuts"))
   (gr_arc (start 27.500343 54.929289) (mid 31.620089 36.845344) (end 43.049312 22.238009)
     (stroke (width 0.2) (type solid)) (layer "Edge.Cuts"))
@@
   (gr_arc (start 43.049312 22.238009) (mid 45.360007 21.585593) (end 47.409169 22.83695)
     (stroke (width 0.2) (type solid)) (layer "Edge.Cuts"))
-  (gr_circle (center 107.5 82.6) (end 109.6 82.6)
-    (stroke (width 0.2) (type solid)) (fill none) (layer "Edge.Cuts"))
   (gr_line (start 31.500343 102.6) (end 108.5 102.6)
     (stroke (width 0.2) (type solid)) (layer "Edge.Cuts"))
   (gr_arc (start 48.272125 24.069378) (mid 48.787365 26.193932) (end 47.724037 28.104047)
     (stroke (width 0.2) (type solid)) (layer "Edge.Cuts"))
-  (gr_circle (center 32.500343 97.6) (end 34.600343 97.6)
-    (stroke (width 0.2) (type solid)) (fill none) (layer "Edge.Cuts"))
-  (gr_circle (center 32.500343 82.6) (end 34.600343 82.6)
-    (stroke (width 0.2) (type solid)) (fill none) (layer "Edge.Cuts"))
   (gr_arc (start 92.275963 28.104047) (mid 91.212635 26.193933) (end 91.727875 24.069378)
     (stroke (width 0.2) (type solid)) (layer "Edge.Cuts"))
-  (gr_circle (center 107.5 97.6) (end 109.6 97.6)
-    (stroke (width 0.2) (type solid)) (fill none) (layer "Edge.Cuts"))
   (gr_text "Designed By \nAlex Eastabrook" (at 111.5 69.5 90) (layer "F.Cu" knockout)
     (effects (font (size 1 1) (thickness 0.25) bold) (justify bottom))
@@
     (effects (font (size 1 1) (thickness 0.25) bold) (justify left bottom))
   )
-  (gr_text "Millennium Machines\nMilo\nLED Ring Light V1" (at 69.5 102) (layer "F.SilkS")
+  (gr_text "Millennium Machines\nMilo\nLED Ring Light V1.1" (at 69.5 102) (layer "F.SilkS")
     (effects (font (size 1 1) (thickness 0.25) bold) (justify bottom))
   )
@@
       17c9725d-a5f6-4260-8856-cfbde7fa71c3
       1a3df542-3d4e-4cf7-8eea-b1c6c8114aa5
-      2658999e-5db4-4eb8-a4dc-ba758de37d6f
-      2886bfdf-121f-48c9-bcba-a49b8c0acde8
       2e3eb74a-94ed-452a-b5a7-7e01474cdf79
       343008fa-da48-4f4e-bb85-da9493eb02be
@@
       4bc0fffb-3fd1-47ef-991f-95242dfaf467
       4c264456-4b29-4ccc-a61c-e56298138cf1
-      4e4b1184-3225-43ce-a8ca-39d0003c9b4f
       4fcc36af-7dbb-46ea-b5fb-802f4015aa76
       5f5489eb-34e6-499a-8746-e176a5807232
@@
       a6bea620-0daf-4da4-b37c-9f2610303b02
       a8570960-391c-40ff-915d-1e643d8b1e49
-      c186b99a-fb74-4d28-bb4b-d7a818205fb5
       c4fe4da6-3d6b-4299-92d9-3d214114869d
       cce99b7c-dd04-4477-92a6-6b9ae4c42659
@@
       d355b036-acd3-48e5-94cb-48e855dac2e4
       dba236ee-6295-4e4b-8979-3291c92441da
-      dc99a841-4321-43ca-8bdb-858db6379ca5
       dfc6e954-94ae-4d3a-b11a-995d66e9c15f
       e9ac34fc-9002-4314-a75d-508589750af1
-      eb60c3ec-cc27-4556-8d2e-21aa776651f1
-      ed1b697d-d6a6-4e0f-8b19-4d8380348bda
       ee75ebba-52c8-4ffa-a930-7fdced1512e9
-      f8c7555b-dc47-4b96-bc26-9c93053dc958
-    )
-  )
+    )
+  )
