File: Milo_Ringlight/KiCad/Milo_RingLight/Milo_RingLight.kicad_sch (KiCad schematic)
At the start: 16 parts, among them J1 Barrel_Jack_MountingPin, J2 MountingHole, J3 MountingHole, J4 MountingHole, J5 MountingHole, J6 Power Connector

Commit message: Continued Work.
Parts:
- J6: footprint Fiducial:Fiducial_0.75mm_Mask2.25mm -> Connector_JST:JST_EH_B2B-EH-A_1x02_P2.50mm_Vertical
Changed lines of the file:
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@@
       (effects (font (size 1.27 1.27)) (justify left))
     )
-    (property "Footprint" "Fiducial:Fiducial_0.75mm_Mask2.25mm" (at 109.22 45.72 0)
+    (property "Footprint" "Connector_JST:JST_EH_B2B-EH-A_1x02_P2.50mm_Vertical" (at 109.22 45.72 0)
       (effects (font (size 1.27 1.27)) hide)
     )
