File: HoverboardDriver/STM32_DualBLDC/EastabrookaBLDC_Project/EastabrookaBLDC_Project.kicad_pcb (KiCad board)
At the start: 2 copper layers, 1 part, among them U2 STM32F407VET6-LQFP100

Commit message: Idk what these deltas are.
Parts:
- added U3: DRV8301DCAR, LocalLibs:SOP50P810X120-57N, F.Cu at (106.7, 48.3)
- added U4: DRV8301DCAR, LocalLibs:SOP50P810X120-57N, F.Cu at (106.7, 71.1)
- moved U2 12.9 mm to (78.7, 61.1)
