File: HoverboardDriver/STM32_DualBLDC/EastabrookaBLDC_Project/EastabrookaBLDC_Project.kicad_sch (KiCad schematic)
At the start: 0 parts

Commit message: Idk what these deltas are.
Other:
- added sheet TI_DRV1 (TI_DRV1.kicad_sch)
- added sheet TI_DRV2 (TI_DRV2.kicad_sch)
Changed lines of the file:
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@@
 (kicad_sch (version 20230121) (generator eeschema)
   (paper "A4")
+  (sheet (at 182.88 57.15) (size 22.86 24.13) (fields_autoplaced)
+    (stroke (width 0.1524) (type solid))
+    (fill (color 0 0 0 0.0000))
+    (property "Sheetname" "TI_DRV1" (at 182.88 56.4384 0)
+      (effects (font (size 1.27 1.27)) (justify left bottom))
+    )
+    (property "Sheetfile" "TI_DRV1.kicad_sch" (at 182.88 81.8646 0)
+      (effects (font (size 1.27 1.27)) (justify left top))
+    )
+    (instances
+      (project "EastabrookaBLDC_Project"
+        (path "/611dd54e-c711-4af1-839a-27cad68a278e" (page "3"))
+      )
+    )
+  )
+  (sheet (at 182.88 91.44) (size 22.86 24.13) (fields_autoplaced)
+    (stroke (width 0.1524) (type solid))
+    (fill (color 0 0 0 0.0000))
+    (property "Sheetname" "TI_DRV2" (at 182.88 90.7284 0)
+      (effects (font (size 1.27 1.27)) (justify left bottom))
+    )
+    (property "Sheetfile" "TI_DRV2.kicad_sch" (at 182.88 116.1546 0)
+      (effects (font (size 1.27 1.27)) (justify left top))
+    )
+    (instances
+      (project "EastabrookaBLDC_Project"
+        (path "/611dd54e-c711-4af1-839a-27cad68a278e" (page "4"))
+      )
+    )
+  )
   (sheet (at 121.92 72.39) (size 38.1 39.37) (fields_autoplaced)
     (stroke (width 0.1524) (type solid))
